File: kicad/current_monitoring_board/current_monitoring_board.kicad_sch (KiCad schematic)
At the start: 44 parts, among them J1 Microsemi_FlashPro-JTAG-10, J2 RJ45_Hanrun_HR911105A_Horizon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, J3 USB_C_Receptacle_USB2.0_16P, J5 CUI_PD-30, Q1 S8050, Q2 S8050, U1 ESP32-WROOM-32E, U2 CH340C, U3 USBLC6-2P6, U4 OPA2333xxD, U5 LAN8720A, U6 AP2112K-3.3, Y2 ASV-50.000MHz

Commit message: first version of pcb
Parts:
- added D6: LED, LED_SMD:LED_0402_1005Metric, symbol Device:LED
- added J5, J6: 1702473, Phoenix connector foot:PHOENIX_1702473, symbol Phoenix Connector:1702473
- added R15: 100k, Resistor_SMD:R_0805_2012Metric, symbol Device:R
- C3: renamed from C1; footprint (none) -> Capacitor_SMD:C_0402_1005Metric
- C4: renamed from C5; footprint (none) -> Capacitor_SMD:C_0402_1005Metric
- C5: renamed from C4; footprint (none) -> Capacitor_SMD:C_0402_1005Metric
- C6: renamed from C7; footprint (none) -> Capacitor_SMD:C_0402_1005Metric
- C7: renamed from C2; footprint (none) -> Capacitor_SMD:C_0402_1005Metric
- C8, C9: footprint (none) -> Capacitor_SMD:C_0402_1005Metric
- renumbered S2 to BOOT_BUTTON1, C6 to C1, C3 to C2, D3 to D1, D4 to D2, D1 to D3, D2 to D4, S1 to EN_BUTTON1, J3 to J1, J5 to J2, J2 to J3, J1 to J4, R6 to R1, R11 to R10, R4 to R11, R14 to R12, R15 to R14, R7 to R2, R8 to R3, R9 to R4, R1 to R5, R2 to R6, R3 to R7, R5 to R8, R12 to R9, RLe to RLe1, RLo to RLo1, U4 to U1, U3 to U2, U6 to U3, U2 to U4, U1 to U6, Y2 to Y1
Connections:
- net +3.3V: now also R15.1
- net GND: now also D6.2 (A), J5.2, J6.2
- net Le_in: now also J6.1
- net Lo_in: now also J5.1
- new net: D6.1 (K), R15.2
Other:
- moved on the sheet: BOOT_BUTTON1, C1, C2, C3, C4, C5, C6, C7, C8, C9, D1, D2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

Commit message: wip
Connections:
- net V_ref: now reaches U6.8 (IO32)
- net V_ref: now also RLe1.1, RLo1.1, U1.1, U1.2 (-), U1.6 (-), U1.7
Changed lines of the file:
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@@
+	)
+	(junction
+		(at 63.5 217.17)
+		(diameter 0)
+		(color 0 0 0 0)
 	)
 	(junction
@@
 	)
 	(junction
+		(at 63.5 171.45)
+		(diameter 0)
+		(color 0 0 0 0)
+	)
+	(junction
 		(at 247.65 38.1)
 		(diameter 0)
@@
 	(wire
 		(pts
-			(xy 58.42 217.17) (xy 74.93 217.17)
+			(xy 58.42 217.17) (xy 63.5 217.17)
 		)
 		(stroke
@@
 	(wire
 		(pts
+			(xy 63.5 171.45) (xy 74.93 171.45)
+		)
+		(stroke
+			(width 0)
+			(type default)
+		)
+	)
+	(wire
+		(pts
 			(xy 31.75 214.63) (xy 31.75 215.9)
 		)
@@
 	(wire
 		(pts
+			(xy 63.5 167.64) (xy 63.5 171.45)
+		)
+		(stroke
+			(width 0)
+			(type default)
+		)
+	)
+	(wire
+		(pts
 			(xy 367.03 78.74) (xy 369.57 78.74)
 		)
@@
 	(wire
 		(pts
+			(xy 222.25 88.9) (xy 223.52 88.9)
+		)
+		(stroke
+			(width 0)
+			(type default)
+		)
+	)
+	(wire
+		(pts
 			(xy 52.07 64.77) (xy 52.07 62.23)
 		)
@@
 	(wire
 		(pts
+			(xy 63.5 212.09) (xy 63.5 217.17)
+		)
+		(stroke
+			(width 0)
+			(type default)
+		)
+	)
+	(wire
+		(pts
 			(xy 367.03 76.2) (xy 370.84 76.2)
 		)
@@
 	(wire
 		(pts
+			(xy 63.5 217.17) (xy 74.93 217.17)
+		)
+		(stroke
+			(width 0)
+			(type default)
+		)
+	)
+	(wire
+		(pts
 			(xy 262.89 44.45) (xy 262.89 38.1)
 		)
@@
 	(wire
 		(pts
-			(xy 58.42 171.45) (xy 74.93 171.45)
+			(xy 58.42 171.45) (xy 63.5 171.45)
 		)
 		(stroke
@@
 		)
 	)
+	(global_label "V_ref"
+		(shape input)
+		(at 223.52 88.9 0)
+		(fields_autoplaced yes)
+		(effects
+			(font
+				(size 1.27 1.27)
+			)
+			(justify left)
+		)
+		(property "Intersheetrefs" "${INTERSHEET_REFS}"
+			(at 231.1619 88.9 0)
+			(hide yes)
+			(show_name no)
+			(do_not_autoplace no)
+			(effects
+				(font
+					(size 1.27 1.27)
+				)
+				(justify left)
+			)
+		)
+	)
 	(global_label "Le_in"
 		(shape input)
@@
 		)
 	)
+	(global_label "V_ref"
+		(shape input)
+		(at 63.5 167.64 90)
+		(fields_autoplaced yes)
+		(effects
+			(font
+				(size 1.27 1.27)
+			)
+			(justify left)
+		)
+		(property "Intersheetrefs" "${INTERSHEET_REFS}"
+			(at 63.5 159.9981 90)
+			(hide yes)
+			(show_name no)
+			(do_not_autoplace no)
+			(effects
+				(font
+					(size 1.27 1.27)
+				)
+				(justify left)
+			)
+		)
+	)
 	(global_label "EN"
 		(shape input)
@@
 			)
 		)
+	)
+	(global_label "V_ref"
+		(shape input)
+		(at 63.5 212.09 90)
+		(fields_autoplaced yes)
+		(effects
+			(font
+				(size 1.27 1.27)
+			)
+			(justify left)
+		)
+		(property "Intersheetrefs" "${INTERSHEET_REFS}"
+			(at 63.5 204.4481 90)
+			(hide yes)
+			(show_name no)
+			(do_not_autoplace no)
+			(effects
+				(font
+					(size 1.27 1.27)
+				)
+				(justify left)
+			)
+		)
